File: Kites/Eagle/Parachute_V1.2.brd (EAGLE design)
At the start: 172.7 x 106.4 mm, 24 parts, among them Q1 MOSFET-NCH, Q2 MOSFET-NCH, U1 ITSYBITSY_5V, X1 MSTBA8

Commit message: Fixed pinout on board causing StopbtnPWN to ground Updated code to have proper breathing animation for each button
Connections:
- new net N$23: JP2.6, U1.RES
- new net N$6: U$1.8, U1.AREF
- net GND: now also U$1.7; no longer U$1.4
- net N$16: now also U$1.9
- net N$17: now also U$1.10
- net N$27: now also U$1.2; no longer U$1.9
- net N$28: now also U$1.3; no longer U$1.8
- net N$29: now also U$1.4; no longer U$1.7
- net N$4: now also U$1.1; no longer U$1.10
Routing:
- net N$6: track 0.00 -> 73.6 mm, vias 0 -> 2
- net N$18: track 89.2 -> 156.0 mm
- net N$5: track 160.4 -> 95.3 mm
- net N$31: track 111.1 -> 66.6 mm
- net N$15: track 86.2 -> 123.4 mm, vias 1 -> 0
- net N$23: track 0.00 -> 37.0 mm
- net N$8: track 92.6 -> 72.8 mm, vias 0 -> 1
- net N$4: track 47.4 -> 66.9 mm
- net N$27: track 106.2 -> 121.8 mm, vias 1 -> 0
- net N$28: track 101.9 -> 116.8 mm
- net N$21: track 166.6 -> 152.9 mm, vias 0 -> 2
- net N$20: track 80.2 -> 68.7 mm, vias 0 -> 1
- net N$22: track 87.2 -> 76.3 mm, vias 0 -> 1
- net N$29: track 96.2 -> 107.1 mm
- net N$13: track 70.3 -> 80.4 mm, vias 0 -> 1
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Other:
- board text added: "DOT: Kites V1.2 7/26/2022 Aaron De Lanty"
- board text removed: "DOT: Kites V1.1 7/26/2022 Aaron De Lanty"
