File: Kites/Eagle/Parachute_V1.5.brd (EAGLE design)
At the start: 172.7 x 106.4 mm, 28 parts, among them Q1 MOSFET-NCH, Q2 MOSFET-NCH, U1 ITSYBITSY_5V, X1 MSTBA8, X2 PHOENIX_508_4PIN, X3 PHOENIX_508_4PIN

Commit message: update
Parts:
- added JP4, JP5: JUMPER-SMT_2_NO_NO-SILK_ROUND, SparkFun-Jumpers:SMT-JUMPER_2_NO_NO-SILK_ROUND
- moved X3 99.9 mm to (99.3, 6.60), turned to 0 degrees
- moved X2 99.2 mm to (127.0, 102.9), turned to 180 degrees
- moved J1 21.0 mm to (-2.54, 68.6), turned to 0 degrees
- moved J2 14.5 mm to (-2.54, 53.3), turned to 0 degrees
Connections:
- removed net N$18: JP10.1, U$1.5, U1.D13
- removed net N$30: J1.4, X2.3
- removed net N$32: J1.2, X2.2
- removed net N$34: J2.4, X3.3
- removed net N$36: J2.2, X3.2
- new net N$12: JP10.3, U$1.5, U1.D12
- net GND: now also JP10.1; no longer JP10.3
- net N$15: now also U1.D13; no longer U1.D12
- net N$24: now also JP4.1
- net N$26: now also JP5.2
- net N$33: now also JP5.1
- net N$35: now also JP4.2
Routing:
- net GND: track 0.00 -> 473.5 mm, vias 0 -> 3
- net N$19: track 0.00 -> 182.6 mm, vias 0 -> 1
- net A3: track 0.00 -> 165.4 mm, vias 0 -> 1
- net N$24: track 0.00 -> 158.6 mm
- net N$35: track 0.00 -> 139.1 mm
- net N$33: track 0.00 -> 137.7 mm, vias 0 -> 1
- net N$26: track 0.00 -> 133.9 mm
- net N$21: track 0.00 -> 129.2 mm, vias 0 -> 2
- net N$28: track 0.00 -> 123.4 mm, vias 0 -> 2
- net 12V: track 0.00 -> 114.8 mm
- net N$29: track 0.00 -> 106.9 mm, vias 0 -> 1
- net N$27: track 0.00 -> 106.8 mm
- net N$3: track 0.00 -> 100.6 mm
- net N$16: track 0.00 -> 98.5 mm, vias 0 -> 1
- net N$17: track 0.00 -> 98.4 mm, vias 0 -> 2
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Other:
- outline, holes or cut-outs redrawn
- board text added: "24V in"
- board text added: "Open Load Bypass"
- board text added: "PWR IN"
- board text added: "TO LEDS"
- board text added: "TO LOAD"
- board text added: "only solder if not using open load module"
