File: Kites/Eagle/Parachute_V1.5.brd (EAGLE design)
At the start: 172.7 x 106.4 mm, 28 parts, among them Q1 MOSFET-NCH, Q2 MOSFET-NCH, U1 ITSYBITSY_5V, X1 MSTBA8, X2 PHOENIX_508_4PIN, X3 PHOENIX_508_4PIN

Commit message: commiting
Parts:
- removed J1, J2: (no value), OMSI_Default_V1:HEADER_PIN_1X05
- removed X2, X3: PHOENIX_508_4PIN, OMSI_Default_V1:PHOENIX_508_4PIN
Connections:
- removed net N$24: J1.1, X2.1
- removed net N$26: J1.5, X2.4
- removed net N$30: J1.4, X2.3
- removed net N$32: J1.2, X2.2
- removed net N$33: J2.5, X3.4
- removed net N$34: J2.4, X3.3
- removed net N$35: J2.1, X3.1
- removed net N$36: J2.2, X3.2
- net A3: no longer J2.3
Other:
- board text removed: "24V"
Changed lines of the file:
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@@
 <text x="20.701" y="73.152" size="1.016" layer="25">Start_PWM</text>
 <text x="33.401" y="73.152" size="1.016" layer="25">Stop_PWM</text>
-<text x="97.155" y="14.224" size="1.778" layer="25" rot="R90">24V</text>
-<text x="112.522" y="13.716" size="1.778" layer="25" rot="R90">GND</text>
-<text x="133.985" y="94.996" size="1.778" layer="25" rot="R270">24V</text>
-<text x="118.618" y="95.504" size="1.778" layer="25" rot="R270">GND</text>
 </plain>
 <attributes>
@@
 <attribute name="VALUE" x="58.42" y="101.6" size="1.778" layer="27" ratio="10" rot="R180"/>
 </element>
-<element name="X2" library="OMSI_Default_V1" library_urn="urn:adsk.eagle:library:40091679" package="PHOENIX_508_4PIN" package3d_urn="urn:adsk.eagle:package:40091802/4" value="PHOENIX_508_4PIN" x="104.14" y="6.35" smashed="yes">
-<attribute name="MF" value="FARNELL" x="104.14" y="6.35" size="1.778" layer="27" display="off"/>
-<attribute name="MPN" value="1757268" x="104.14" y="6.35" size="1.778" layer="27" display="off"/>
-<attribute name="OC_FARNELL" value="3705195" x="104.14" y="6.35" size="1.778" layer="27" display="off"/>
-<attribute name="OC_NEWARK" value="71C4163" x="104.14" y="6.35" size="1.778" layer="27" display="off"/>
-<attribute name="POPULARITY" value="9" x="104.14" y="6.35" size="1.778" layer="27" display="off"/>
-</element>
-<element name="X3" library="OMSI_Default_V1" library_urn="urn:adsk.eagle:library:40091679" package="PHOENIX_508_4PIN" package3d_urn="urn:adsk.eagle:package:40091802/4" value="PHOENIX_508_4PIN" x="126.746" y="102.616" smashed="yes" rot="R180">
-<attribute name="MF" value="FARNELL" x="126.746" y="102.616" size="1.778" layer="27" rot="R180" display="off"/>
-<attribute name="MPN" value="1757268" x="126.746" y="102.616" size="1.778" layer="27" rot="R180" display="off"/>
-<attribute name="OC_FARNELL" value="3705195" x="126.746" y="102.616" size="1.778" layer="27" rot="R180" display="off"/>
-<attribute name="OC_NEWARK" value="71C4163" x="126.746" y="102.616" size="1.778" layer="27" rot="R180" display="off"/>
-<attribute name="POPULARITY" value="9" x="126.746" y="102.616" size="1.778" layer="27" rot="R180" display="off"/>
-</element>
-<element name="J1" library="OMSI_Default_V1" library_urn="urn:adsk.eagle:library:40091679" package="HEADER_PIN_1X05" package3d_urn="urn:adsk.eagle:package:40091793/3" value="" x="6.35" y="49.53" smashed="yes" rot="R180">
-<attribute name="NAME" x="7.62" y="48.133" size="0.6096" layer="25" font="vector" ratio="20" rot="R180"/>
-<attribute name="VALUE" x="7.62" y="51.562" size="0.6096" layer="27" font="vector" ratio="20" rot="R180"/>
-</element>
-<element name="J2" library="OMSI_Default_V1" library_urn="urn:adsk.eagle:library:40091679" package="HEADER_PIN_1X05" package3d_urn="urn:adsk.eagle:package:40091793/3" value="" x="6.35" y="64.77" smashed="yes" rot="R180">
-<attribute name="NAME" x="7.62" y="63.373" size="0.6096" layer="25" font="vector" ratio="20" rot="R180"/>
-<attribute name="VALUE" x="7.62" y="66.802" size="0.6096" layer="27" font="vector" ratio="20" rot="R180"/>
-</element>
 </elements>
 <signals>
@@
 <contactref element="JP12" pad="3"/>
 <contactref element="JP3" pad="4"/>
-<contactref element="J2" pad="3"/>
 <wire x1="112.649" y1="29.083" x2="110.109" y2="33.782" width="0" layer="19" extent="1-1"/>
 <wire x1="59.69" y1="24.13" x2="110.109" y2="33.782" width="0" layer="19" extent="1-1"/>
-<wire x1="1.27" y1="64.77" x2="59.69" y2="24.13" width="0" layer="19" extent="1-1"/>
 </signal>
 <signal name="N$13">
@@
 <wire x1="59.69" y1="6.35" x2="87.249" y2="29.083" width="0" layer="19" extent="1-1"/>
 </signal>
-<signal name="N$24">
-<contactref element="X2" pad="1"/>
-<contactref element="J1" pad="1"/>
-<wire x1="96.52" y1="11.43" x2="6.35" y2="49.53" width="0" layer="19" extent="1-1"/>
-</signal>
-<signal name="N$26">
-<contactref element="X2" pad="4"/>
-<contactref element="J1" pad="5"/>
-<wire x1="111.76" y1="11.43" x2="-3.81" y2="49.53" width="0" layer="19" extent="1-1"/>
-</signal>
-<signal name="N$30">
-<contactref element="X2" pad="3"/>
-<contactref element="J1" pad="4"/>
-<wire x1="106.68" y1="11.43" x2="-1.27" y2="49.53" width="0" layer="19" extent="1-1"/>
-</signal>
-<signal name="N$32">
-<contactref element="X2" pad="2"/>
-<contactref element="J1" pad="2"/>
-<wire x1="101.6" y1="11.43" x2="3.81" y2="49.53" width="0" layer="19" extent="1-1"/>
-</signal>
-<signal name="N$33">
-<contactref element="X3" pad="4"/>
-<contactref element="J2" pad="5"/>
-<wire x1="119.126" y1="97.536" x2="-3.81" y2="64.77" width="0" layer="19" extent="1-1"/>
-</signal>
-<signal name="N$34">
-<contactref element="J2" pad="4"/>
-<contactref element="X3" pad="3"/>
-<wire x1="124.206" y1="97.536" x2="-1.27" y2="64.77" width="0" layer="19" extent="1-1"/>
-</signal>
-<signal name="N$35">
-<contactref element="X3" pad="1"/>
-<contactref element="J2" pad="1"/>
-<wire x1="134.366" y1="97.536" x2="6.35" y2="64.77" width="0" layer="19" extent="1-1"/>
-</signal>
-<signal name="N$36">
-<contactref element="X3" pad="2"/>
-<contactref element="J2" pad="2"/>
-<wire x1="129.286" y1="97.536" x2="3.81" y2="64.77" width="0" layer="19" extent="1-1"/>
-</signal>
 </signals>
