File: Kites/Eagle/Parachute_V1.5.sch (EAGLE design)
At the start: 28 parts, among them Q1 MOSFET-NCH, Q2 MOSFET-NCH, U1 ITSYBITSY_5V, X1 MSTBA8, X2 PHOENIX_508_4PIN, X3 PHOENIX_508_4PIN

Commit message: update
Parts:
- added JP4, JP5: JUMPER-SMT_2_NO_NO-SILK_ROUND, SparkFun-Jumpers:JUMPER-SMT_2_NO_NO-SILK_ROUND
Connections:
- removed net N$18: JP10.1, U$1.5, U1.D13
- removed net N$30: J1.4, X2-3.1
- removed net N$32: J1.2, X2-2.1
- removed net N$34: J2.4, X3-3.1
- removed net N$36: J2.2, X3-2.1
- new net N$12: JP10.3, U$1.5, U1.D12
- net GND: now also JP10.1; no longer JP10.3
- net N$15: now also U1.D13; no longer U1.D12
- net N$24: now also JP4.1
- net N$26: now also JP5.2
- net N$33: now also JP5.1
- net N$35: now also JP4.2
Other:
- moved on the sheet: J2, X2-1, X2-2, X2-3, X2-4, X3-1, X3-2, X3-3, X3-4
