File: Kites/Eagle/Parachute_V1.5(openloadsensor).sch (EAGLE design)
At the start: 28 parts, among them Q1 MOSFET-NCH, Q2 MOSFET-NCH, U1 ITSYBITSY_5V, X1 MSTBA8, X2 PHOENIX_508_4PIN, X3 PHOENIX_508_4PIN

Commit message: commiting
Changed lines of the file:
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@@
 <attribute name="VALUE" x="127" y="197.866" size="1.778" layer="96" rot="R180" align="bottom-center"/>
 </instance>
-<instance part="GND10" gate="1" x="152.4" y="147.32" smashed="yes">
-<attribute name="VALUE" x="149.86" y="144.78" size="1.778" layer="96"/>
+<instance part="GND10" gate="1" x="157.48" y="213.36" smashed="yes">
+<attribute name="VALUE" x="154.94" y="210.82" size="1.778" layer="96"/>
 </instance>
 <instance part="JP1" gate="G$1" x="15.24" y="111.76" smashed="yes" rot="R180">
@@
 <pinref part="JP10" gate="G$1" pin="3"/>
 <pinref part="GND10" gate="1" pin="GND"/>
-<wire x1="157.48" y1="149.86" x2="152.4" y2="149.86" width="0.1524" layer="91"/>
+<wire x1="157.48" y1="149.86" x2="157.48" y2="215.9" width="0.1524" layer="91"/>
 </segment>
 <segment>
