File: Prairie_Dogs/Eagle/Prairie_Dogs_V1.3.brd (EAGLE design)
At the start: 172.7 x 106.4 mm, 19 parts, among them Q1 MOSFET-NCH, Q2 MOSFET-NCH, U1 ITSYBITSY_5V

Commit message: Documentation
Started Documentation
Parts:
- added CALIBRATION_BTN: MSTBA2, th_libraries:MSTBA2
- moved HAPP_STARTBUTTON 14.0 mm to (96.0, 101.6)
Connections:
- new net N$14: CALIBRATION_BTN.2, U1.D5
- net GND: now also CALIBRATION_BTN.1
Routing:
- net N$14: track 0.00 -> 73.5 mm
- net N$5: track 83.9 -> 66.1 mm, vias 0 -> 1
- net N$1: track 97.5 -> 86.1 mm
- net N$10: track 66.2 -> 59.6 mm
- net N$12: track 88.0 -> 82.0 mm, vias 0 -> 1
- net 12V: track 280.1 -> 274.7 mm
- net N$2: track 62.8 -> 57.5 mm
- net N$3: track 93.1 -> 90.9 mm
- net GND: track 402.2 -> 401.1 mm
Other:
- board text added: "DOT: Prairie Dogs V1.3 11/11/2022 Aaron De Lanty"
- board text removed: "DOT: Prairie Dogs V1.2 9/30/2022 Aaron De Lanty"
