File: Prairie_Dogs/Eagle/Prairie_Dogs_V1.3.brd (EAGLE design)
At the start: 172.7 x 106.4 mm, 19 parts, among them Q1 MOSFET-NCH, U1 ITSYBITSY_5V, X1 PHOENIX_508_3PIN

Commit message: changed the direction of lights and logic
instead of having one array that is broken up into pointers and then manually changed we break up the large array into smaller ones and then address each one seperately
Connections:
- net N$9 renamed D11
Changed lines of the file:
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@@
 <wire x1="55.88" y1="12.7" x2="32.004" y2="36.576" width="0.4064" layer="1"/>
 </signal>
-<signal name="N$9">
+<signal name="D11">
 <contactref element="U1" pad="D11"/>
 <contactref element="10K" pad="2"/>
