File: Rooftop-Reflector/Eagle/rooftop_reflector.brd (EAGLE design)
At the start: 172.7 x 106.4 mm, 18 parts, among them Q1 MOSFET-NCH, Q4 MOSFET-NCH, U1 ADAFRUIT_LEONARDO, X1 MSTBA4

Commit message: Updated Btn calls and added Pulse function
Parts:
- removed 5VIN: MSTBA2, con-phoenix-508:MSTBA2
- added 5V: L7805ABD2T-TR, SamacSys_Parts:D2PAK-STB35NF10T4
- added 9V: BA17809FP-E2, SamacSys_Parts:BA17809FPE2
Connections:
- net N$1 renamed D9
- net N$3 renamed SRT_PWM
- net N$5 renamed D5
- net N$6 renamed LZR_CTL
- removed net N$9: U1.VIN, X1.4
- new net 9V: 9V.3, LASER_CTL.1, LASER_CTL.3
- net 12V: now also 5V.1, 9V.1
- net 5V: now also 5V.3, U1.VIN, X1.4; no longer 5VIN.1, LASER_CTL.1, LASER_CTL.3, TP2.TP-2
- net GND: now also 5V.4, 9V.2; no longer 5VIN.2, TP1.TP-2
Routing:
- net 9V: track 0.00 -> 103.1 mm, vias 0 -> 2
- net 5V: track 137.6 -> 103.9 mm, vias 1 -> 0
- net N$9: track 18.0 -> 0.00 mm
- net 12V: track 102.6 -> 116.2 mm, vias 0 -> 1
- net SRT_PWM: vias 0 -> 1
