File: Bird_Beaks/Eagle/bird_beaks 2.0.brd (EAGLE design)
At the start: 172.7 x 106.4 mm, 23 parts, among them Q1 MOSFET-NCH, Q2 MOSFET-NCH, Q3 MOSFET-NCH, U1 ITSYBITSY_5V, X1 MSTBA4, X2 MSTBA4, X3 MSTBA4, X4 MSTBA2, X5 MSTBA2, X6 MSTBA2, X7 MSTBA2

Commit message: board edits
Parts:
- added 10K10, 10K11, 10K3, 10K4, 10K5, 10K6, 10K7, 10K8, 10K9: (no value), adafruit:M0805
- added Q10, Q11, Q12, Q4, Q5, Q6, Q7, Q8, Q9: MOSFET-NCH, th_ds_libraries:SO-8_POWER_PAK
- added U$1: TLC59711, OMSI_Default_V1:ADAFRUIT_TLC59711
Connections:
- removed net N$3 (its old number): U1.D5, U1.RES
- new net D1: 10K3.2
- new net D14: 10K10.2
- new net D15: 10K11.2
- new net D2: 10K4.2
- new net D4: 10K6.2
- new net D5: 10K7.2
- new net D6: 10K8.2
- new net D8: 10K9.2
- new net N$12: 10K5.1, Q6.G
- new net N$13: Q6.D1, U$1.R0
- new net N$14: 10K6.1, Q7.G
- new net N$15: Q7.D1
- new net N$16: 10K7.1, Q8.G
- new net N$17: Q8.D1
- new net N$18: 10K8.1, Q9.G
- new net N$19: Q9.D1
- new net N$20: 10K9.1, Q10.G
- new net N$21: Q10.D1
- new net N$22: 10K10.1, Q11.G
- new net N$23: Q11.D1
- new net N$24: 10K11.1, Q12.G
- new net N$25: Q12.D1
- new net N$4: 10K3.1, Q4.G
- new net N$5: Q4.D1
- new net N$6: 10K4.1, Q5.G
- new net N$9: Q5.D1
- new net SCL: U$1.CI, U$1.CO, U1.SCL
- new net SDA: U$1.DI, U$1.DO, U1.SDA
- new net V+: 10K5.2, U$1.P$10, U$1.P$11, U$1.P$15, U$1.P$16, U$1.P$17, U$1.P$20, U$1.P$24, U$1.P$25, U$1.P$28, U$1.P$29, U$1.P$3, U$1.P$32, U$1.P$33, U$1.P$9
- net 5V: now also U$1.P$2, U$1.P$21
- net GND: now also Q10.S, Q11.S, Q12.S, Q4.S, Q5.S, Q6.S, Q7.S, Q8.S, Q9.S, U$1.P$1, U$1.P$22
Routing:
- net GND: track 0.00 -> 421.9 mm, vias 0 -> 2
- net N$3: track 56.6 -> 0.00 mm, vias 1 -> 0
- net N$3 (its old number): track 29.2 -> 0.00 mm
- net NUT_LIGHT: track 79.3 -> 74.8 mm, vias 0 -> 1
- net N$8: vias 1 -> 2
- removed copper zone on layer 1, net GND
- removed copper zone on layer 16, net GND
