File: Bird_Beaks/Eagle/Light module.brd (EAGLE design)
At the start: 180 x 180 mm, 6 parts

Commit message: updates
Parts:
- removed FROM_MAIN, LEDS: MSTBA2, th_libraries:MSTBA2
- added PWR_IN, TO_LEDS: MSTBA2, th_libraries:MSTBA2
- moved S4 180.1 mm to (119.4, 4.45)
- moved S3 166.5 mm to (8.89, 4.45)
- moved S8 130.8 mm to (63.5, 55.9)
- moved S2 84.9 mm to (63.5, -55.9)
Connections:
- removed net N$1: FROM_MAIN.1, LEDS.1
- removed net N$2: FROM_MAIN.2, LEDS.2
- new net 12V: PWR_IN.2, TO_LEDS.2
- net GND: now also PWR_IN.1, TO_LEDS.1
Routing:
- net GND: track 495.9 -> 1.32 mm
- net N$2: track 185.3 -> 0.00 mm
- net N$1: track 128.7 -> 0.00 mm
- net 12V: track 0.00 -> 54.8 mm
- added copper zone on layer 16, net GND
Other:
- board size 180 x 180 mm -> 127 x 127 mm
- board text added: "DOT: Bird Beaks Light Module V2.0 8/16/2022 Aaron De Lanty"
- board text removed: "DOT: Bird Beaks Light Module V1.0 8/16/2022 Aaron De Lanty"

Commit message: update
Parts:
- removed PWR_IN, TO_LEDS: MSTBA2, th_libraries:MSTBA2
- added J1, J10, J2, J3, J4, J5, J6, J7, J8, J9: (no value), OMSI_Default_V1:HEADER_PIN_1X03
- added X1: PHOENIX_508_3PIN, OMSI_Default_V1:PHOENIX_508_3PIN
Connections:
- removed net 12V: PWR_IN.2, TO_LEDS.2
- new net 5V: J1.1, J10.1, J2.1, J3.1, J4.1, J5.1, J6.1, J7.1, J8.1, J9.1, X1.1
- new net N$11: J6.2, J7.2
- new net N$14: J8.2, J9.2
- new net N$2: J1.2, X1.2
- new net N$5: J2.2, J3.2
- new net N$8: J4.2, J5.2
- net GND: now also J1.3, J10.3, J2.3, J3.3, J4.3, J5.3, J6.3, J7.3, J8.3, J9.3, X1.3; no longer PWR_IN.1, TO_LEDS.1
Routing:
- net GND: track 1.32 -> 355.4 mm
- net 5V: track 0.00 -> 268.7 mm
- net N$2: track 0.00 -> 79.0 mm
- net 12V: track 54.8 -> 0.00 mm
- net N$14: track 0.00 -> 23.6 mm
- net N$8: track 0.00 -> 22.9 mm
- net N$5: track 0.00 -> 21.7 mm
- net N$11: track 0.00 -> 20.4 mm
- removed copper zone on layer 16, net GND
Other:
- board text added: "5v"
- board text added: "DIN"
- board text added: "DO"
- board text added: "↑"
- board text added: "↓"
- board text removed: "12V"
