File: Bird_Beaks/Eagle/Light module.sch (EAGLE design)
At the start: 6 parts

Commit message: update
Parts:
- removed PWR_IN, TO_LEDS: MSTBA2, th_libraries:MSTBA2
- added J1, J10, J2, J3, J4, J5, J6, J7, J8, J9: (no value), OMSI_Default_V1:JST_CONN_03
- added X1: PHOENIX_508_3PIN, OMSI_Default_V1:PHOENIX_508_3PIN
Connections:
- removed net 12V: PWR_IN-2.1, TO_LEDS-2.1
- new net 5V: J1.1, J10.1, J2.1, J3.1, J4.1, J5.1, J6.1, J7.1, J8.1, J9.1, X1-1.1
- new net N$11: J6.2, J7.2
- new net N$14: J8.2, J9.2
- new net N$2: J1.2, X1-2.1
- new net N$5: J2.2, J3.2
- new net N$8: J4.2, J5.2
- net GND: now also J1.3, J10.3, J2.3, J3.3, J4.3, J5.3, J6.3, J7.3, J8.3, J9.3, X1-3.1; no longer PWR_IN-1.1, TO_LEDS-1.1
