File: Kites/Eagle/Archive/Parachute_V1.2.brd (EAGLE design)
At the start: 172.7 x 106.4 mm, 28 parts, among them Q1 MOSFET-NCH, Q2 MOSFET-NCH, U1 ITSYBITSY_5V, X1 MSTBA8, X2 PHOENIX_508_4PIN, X3 PHOENIX_508_4PIN

Commit message: graphics
Parts:
- removed J1, J2: (no value), OMSI_Default_V1:HEADER_PIN_1X05
- removed X2, X3: PHOENIX_508_4PIN, OMSI_Default_V1:PHOENIX_508_4PIN
- moved FAN_POWER 0.89 mm to (95.2, 101.6)
Connections:
- removed net A3: J2.3, JP12.3, JP3.4, U1.A3
- removed net N$24: J1.1, X2.1
- removed net N$26: J1.5, X2.4
- removed net N$30: J1.4, X2.3
- removed net N$32: J1.2, X2.2
- removed net N$33: J2.5, X3.4
- removed net N$34: J2.4, X3.3
- removed net N$35: J2.1, X3.1
- removed net N$36: J2.2, X3.2
- new net N$12: JP12.3, JP3.4, U1.A3
Routing:
- net GND: track 0.00 -> 460.5 mm, vias 0 -> 1
- net N$19: track 0.00 -> 195.3 mm, vias 0 -> 1
- net N$21: track 0.00 -> 134.1 mm, vias 0 -> 2
- net N$18: track 0.00 -> 126.9 mm, vias 0 -> 1
- net N$27: track 0.00 -> 124.3 mm
- net N$15: track 0.00 -> 119.9 mm
- net N$28: track 0.00 -> 116.3 mm, vias 0 -> 2
- net N$29: track 0.00 -> 115.7 mm, vias 0 -> 1
- net 12V: track 0.00 -> 114.8 mm
- net 5V: track 0.00 -> 104.0 mm
- net N$17: track 0.00 -> 97.4 mm
- net N$16: track 0.00 -> 95.9 mm, vias 0 -> 1
- net N$5: track 0.00 -> 94.9 mm
- net N$3: track 0.00 -> 92.7 mm
- net N$22: track 0.00 -> 77.4 mm, vias 0 -> 1
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Other:
- board text removed: "24V"
