File: Kites/Eagle/Archive/Parachute_V1.2.sch (EAGLE design)
At the start: 28 parts, among them Q1 MOSFET-NCH, Q2 MOSFET-NCH, U1 ITSYBITSY_5V, X1 MSTBA8, X2 PHOENIX_508_4PIN, X3 PHOENIX_508_4PIN

Commit message: graphics
Parts:
- removed J1, J2: (no value), OMSI_Default_V1:JST_CONN_05
- removed X2, X3: PHOENIX_508_4PIN, OMSI_Default_V1:PHOENIX_508_4PIN
Connections:
- removed net A3: J2.3, JP12.3, JP3.4, U1.A3
- removed net N$24: J1.1, X2-1.1
- removed net N$26: J1.5, X2-4.1
- removed net N$30: J1.4, X2-3.1
- removed net N$32: J1.2, X2-2.1
- removed net N$33: J2.5, X3-4.1
- removed net N$34: J2.4, X3-3.1
- removed net N$35: J2.1, X3-1.1
- removed net N$36: J2.2, X3-2.1
- new net N$12: JP12.3, JP3.4, U1.A3
Changed lines of the file:
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@@
 <part name="Q2" library="th_ds_libraries" deviceset="MOSFET-NCH" device="" package3d_urn="urn:adsk.eagle:package:26281953/1"/>
 <part name="X1" library="con-phoenix-508" library_urn="urn:adsk.eagle:library:176" deviceset="MSTBA8" device="" package3d_urn="urn:adsk.eagle:package:9620/1"/>
-<part name="X2" library="OMSI_Default_V1" library_urn="urn:adsk.eagle:library:40091679" deviceset="PHOENIX_508_4PIN" device="" package3d_urn="urn:adsk.eagle:package:40091802/4"/>
-<part name="X3" library="OMSI_Default_V1" library_urn="urn:adsk.eagle:library:40091679" deviceset="PHOENIX_508_4PIN" device="" package3d_urn="urn:adsk.eagle:package:40091802/4"/>
-<part name="J1" library="OMSI_Default_V1" library_urn="urn:adsk.eagle:library:40091679" deviceset="JST_CONN_05" device="" package3d_urn="urn:adsk.eagle:package:40091793/3"/>
-<part name="J2" library="OMSI_Default_V1" library_urn="urn:adsk.eagle:library:40091679" deviceset="JST_CONN_05" device="" package3d_urn="urn:adsk.eagle:package:40091793/3"/>
 </parts>
 <sheets>
@@
 <attribute name="NAME" x="196.469" y="207.264" size="1.778" layer="95" rot="R90"/>
 </instance>
-<instance part="X2" gate="-1" x="266.7" y="93.98" smashed="yes">
-<attribute name="NAME" x="260.096" y="94.869" size="1.778" layer="95" rot="R180"/>
-</instance>
-<instance part="X2" gate="-2" x="266.7" y="88.9" smashed="yes">
-<attribute name="NAME" x="260.096" y="89.789" size="1.778" layer="95" rot="R180"/>
-</instance>
-<instance part="X2" gate="-3" x="266.7" y="83.82" smashed="yes">
-<attribute name="NAME" x="260.096" y="84.709" size="1.778" layer="95" rot="R180"/>
-</instance>
-<instance part="X2" gate="-4" x="266.7" y="78.74" smashed="yes">
-<attribute name="NAME" x="260.096" y="79.629" size="1.778" layer="95" rot="R180"/>
-</instance>
-<instance part="X3" gate="-1" x="355.6" y="78.74" smashed="yes" rot="R180">
-<attribute name="NAME" x="362.204" y="77.851" size="1.778" layer="95"/>
-</instance>
-<instance part="X3" gate="-2" x="355.6" y="83.82" smashed="yes" rot="R180">
-<attribute name="NAME" x="362.204" y="82.931" size="1.778" layer="95"/>
-</instance>
-<instance part="X3" gate="-3" x="355.6" y="88.9" smashed="yes" rot="R180">
-<attribute name="NAME" x="362.204" y="88.011" size="1.778" layer="95"/>
-</instance>
-<instance part="X3" gate="-4" x="355.6" y="93.98" smashed="yes" rot="R180">
-<attribute name="NAME" x="362.204" y="93.091" size="1.778" layer="95"/>
-</instance>
-<instance part="J1" gate="G$1" x="292.1" y="86.36" smashed="yes" rot="R180">
-<attribute name="VALUE" x="294.64" y="96.266" size="1.778" layer="96" font="vector" rot="R180"/>
-<attribute name="NAME" x="294.64" y="78.232" size="1.778" layer="95" font="vector" rot="R180"/>
-</instance>
-<instance part="J2" gate="G$1" x="314.96" y="86.36" smashed="yes">
-<attribute name="VALUE" x="312.42" y="76.454" size="1.778" layer="96" font="vector"/>
-<attribute name="NAME" x="312.42" y="94.488" size="1.778" layer="95" font="vector"/>
-</instance>
 </instances>
 <busses>
@@
 </segment>
 </net>
-<net name="A3" class="0">
+<net name="N$12" class="0">
 <segment>
 <pinref part="U1" gate="G$1" pin="A3"/>
@@
 <wire x1="60.96" y1="30.48" x2="60.96" y2="144.78" width="0.1524" layer="91"/>
 <junction x="60.96" y="144.78"/>
-<wire x1="60.96" y1="30.48" x2="73.66" y2="30.48" width="0.1524" layer="91"/>
-<junction x="60.96" y="30.48"/>
-<label x="73.66" y="30.48" size="1.778" layer="95"/>
-</segment>
-<segment>
-<pinref part="J2" gate="G$1" pin="3"/>
-<wire x1="322.58" y1="86.36" x2="330.2" y2="86.36" width="0.1524" layer="91"/>
-<wire x1="330.2" y1="86.36" x2="330.2" y2="66.04" width="0.1524" layer="91"/>
-<label x="330.2" y="66.04" size="1.778" layer="95"/>
 </segment>
 </net>
@@
 </segment>
 </net>
-<net name="N$24" class="0">
-<segment>
-<pinref part="X2" gate="-1" pin="1"/>
-<pinref part="J1" gate="G$1" pin="1"/>
-<wire x1="271.78" y1="93.98" x2="284.48" y2="93.98" width="0.1524" layer="91"/>
-<wire x1="284.48" y1="93.98" x2="284.48" y2="91.44" width="0.1524" layer="91"/>
-</segment>
-</net>
-<net name="N$26" class="0">
-<segment>
-<pinref part="X2" gate="-4" pin="1"/>
-<pinref part="J1" gate="G$1" pin="5"/>
-<wire x1="271.78" y1="78.74" x2="284.48" y2="78.74" width="0.1524" layer="91"/>
-<wire x1="284.48" y1="78.74" x2="284.48" y2="81.28" width="0.1524" layer="91"/>
-</segment>
-</net>
-<net name="N$30" class="0">
-<segment>
-<pinref part="X2" gate="-3" pin="1"/>
-<pinref part="J1" gate="G$1" pin="4"/>
-<wire x1="271.78" y1="83.82" x2="284.48" y2="83.82" width="0.1524" layer="91"/>
-</segment>
-</net>
-<net name="N$32" class="0">
-<segment>
-<pinref part="X2" gate="-2" pin="1"/>
-<pinref part="J1" gate="G$1" pin="2"/>
-<wire x1="271.78" y1="88.9" x2="284.48" y2="88.9" width="0.1524" layer="91"/>
-</segment>
-</net>
-<net name="N$33" class="0">
-<segment>
-<pinref part="X3" gate="-4" pin="1"/>
-<pinref part="J2" gate="G$1" pin="5"/>
-<wire x1="350.52" y1="93.98" x2="322.58" y2="93.98" width="0.1524" layer="91"/>
-<wire x1="322.58" y1="93.98" x2="322.58" y2="91.44" width="0.1524" layer="91"/>
-</segment>
-</net>
-<net name="N$34" class="0">
-<segment>
-<pinref part="J2" gate="G$1" pin="4"/>
-<pinref part="X3" gate="-3" pin="1"/>
-<wire x1="322.58" y1="88.9" x2="350.52" y2="88.9" width="0.1524" layer="91"/>
-</segment>
-</net>
-<net name="N$35" class="0">
-<segment>
-<pinref part="X3" gate="-1" pin="1"/>
-<pinref part="J2" gate="G$1" pin="1"/>
-<wire x1="350.52" y1="78.74" x2="322.58" y2="78.74" width="0.1524" layer="91"/>
-<wire x1="322.58" y1="78.74" x2="322.58" y2="81.28" width="0.1524" layer="91"/>
-</segment>
-</net>
-<net name="N$36" class="0">
-<segment>
-<pinref part="X3" gate="-2" pin="1"/>
-<pinref part="J2" gate="G$1" pin="2"/>
-<wire x1="350.52" y1="83.82" x2="322.58" y2="83.82" width="0.1524" layer="91"/>
-</segment>
-</net>
